File: Hardware/EV-ESP32-energimonitor.kicad_sch (KiCad schematic)
At the start: 78 parts, among them J1 Screw_Terminal_01x02, J2 Conn_01x02_Pin, J3 RJ22, J4 Conn_01x01_Pin, J5 Conn_01x06_Pin, J6 Conn_01x06_Pin, J7 Conn_01x06_Pin, J8 Conn_01x06_Pin, Q1 BC547, Q10 AO3401A, Q11 BC547, Q2 IRF4905, Q4 S8050_NPN, Q5 S8050_NPN, Q6 S8050_NPN, Q7 S8050_NPN, Q8 BC547, Q9 NPN, SW1 SW_Push, SW2 SW_MEC_5E, SW2 SW_Push, SW3 SW_Push, SW4 SW_Push, U1 74HC14, U1 ER_OLEDM0.91_1x-I2C, U2 74HC14, U5 74HC14

Commit message: HW: Prepared for autoroute
Parts:
- removed C1, C11, C12: 100n, symbol Device:C
- removed C10: C_Polarized, symbol Device:C_Polarized
- removed C2: 100nf, Capacitor_SMD:C_0402_1005Metric, symbol Local_Device_Library:C10nf
- removed C3, C9: 1uF, symbol Device:C
- removed C4: 47nf, Capacitor_SMD:C_0402_1005Metric, symbol Local_Device_Library:C10nf
- removed C5: 10uF, symbol Device:C
- removed D1, D2, D3: 1N4148WS, Diode_SMD:D_SOD-323F, symbol Local_Diode_Library:1N4148WS
- removed J2: Conn_01x02_Pin, symbol Connector:Conn_01x02_Pin
- removed J4: Conn_01x01_Pin, symbol Connector:Conn_01x01_Pin
- removed J5, J6, J7, J8: Conn_01x06_Pin, symbol Connector:Conn_01x06_Pin
- removed PS1: RAC04-05SGA, Converter_ACDC:Converter_ACDC_RECOM_RAC04-xxSGx_THT, symbol Converter_ACDC:RAC04-05SGA
- removed Q1, Q11, Q8: BC547, Package_TO_SOT_THT:TO-92_Inline, symbol Transistor_BJT:BC547
- removed Q10: AO3401A, Package_TO_SOT_SMD:SOT-23, symbol Transistor_FET:AO3401A
- removed Q2: IRF4905, Package_TO_SOT_THT:TO-220-3_Vertical, symbol Transistor_FET:IRF4905
- removed Q5, Q6, Q7: S8050_NPN, Package_TO_SOT_SMD:SOT-23, symbol Local_Transistor_BJT_Library:S8050_NPN
- removed Q9: NPN, symbol Simulation_SPICE:NPN
- removed R1: 47K, symbol Device:R
- removed R1, R11, R12, R2: R10K, Resistor_SMD:R_0402_1005Metric, symbol Local_Device_Library:R10K
- removed R10, R13: R180, Resistor_SMD:R_0805_2012Metric, symbol Local_Device_Library:R180
- removed R2: 68K, symbol Device:R
- removed R23: 4.7K, symbol Device:R
- removed R3, R4, R7 (x2): 100K, symbol Device:R
- removed R3: 220K, symbol Device:R
- removed R4, R5, R6 (x2), R7, R8: R4.7K, Resistor_SMD:R_0402_1005Metric, symbol Local_Device_Library:R4.7K
- removed R5: 330K -> 390K, symbol Device:R
- removed R6: 2,2K, symbol Device:R
- removed R9: 10K, symbol Device:R
- removed SW2: SW_MEC_5E, symbol Switch:SW_MEC_5E
- removed U1: ER_OLEDM0.91_1x-I2C, Display:ER_OLEDM0.91_1x-I2C, symbol Display_Graphic:ER_OLEDM0.91_1x-I2C
- added C10, C11, C12, C13, C18: C100nf, Capacitor_SMD:C_0402_1005Metric, symbol Local_Device_Library:C100nf
- added C14: C1uf, Capacitor_SMD:C_0402_1005Metric, symbol Local_Device_Library:C1uf
- added C15: C47nf, Capacitor_SMD:C_0603_1608Metric, symbol Local_Device_Library:C47nf
- added C16, C17, C9: C10uf, Capacitor_SMD:C_0603_1608Metric, symbol Local_Device_Library:C10uf
- added D5, D6, D7: 1N4148WS, Diode_SMD:D_SOD-323F, symbol Local_Diode_Library:1N4148WS
- added J1, J3, J4, J5: Pin_Header_1x6, Local_Connectors:PinHeader_1x06_P_0,1in_Vertical, symbol Local_Connectors_Library:Pin_Header_1x6
- added J2: Conn_2P_Horizontal, Connector_PinHeader_2.54mm:PinHeader_1x02_P2.54mm_Horizontal, symbol Local_Connectors_Library:Conn_2P_Horizontal
- added J6: Conn_1P, Connector_PinHeader_2.54mm:PinHeader_1x01_P2.54mm_Vertical, symbol Local_Connectors_Library:Conn_1P
- added PS1: RAC02-05SC, Local_Misckllaneous_Library:CONV_RAC02-05SC, symbol Local_Miscellaneous_Library:RAC02-05SC
- added Q1, Q2, Q3: S8050_NPN, Package_TO_SOT_SMD:SOT-23, symbol Local_Transistor_BJT_Library:S8050_NPN
- added Q9: AO3401A, Package_TO_SOT_SMD:SOT-23, symbol Local_Transistor_BJT_Library:AO3401A
- added R1, R4: R47K, Resistor_SMD:R_0603_1608Metric, symbol Local_Device_Library:R47K
- added R10, R13, R17: R4.7K, Resistor_SMD:R_0402_1005Metric, symbol Local_Device_Library:R4.7K
- added R11, R12, R5, R7: R100K, Resistor_SMD:R_0402_1005Metric, symbol Local_Device_Library:R100K
- added R14, R15, R16: R10K, Resistor_SMD:R_0402_1005Metric, symbol Local_Device_Library:R10K
- added R18: R2,1K, Local_Resistor_Library:R_Axial_DIN0207_L6.3mm_D2.5mm_P10.16mm_Horizontal, symbol Device:R
- added R2, R9: R68K, Resistor_SMD:R_0603_1608Metric, symbol Local_Device_Library:R68K
- added R20, R21: R1K, Resistor_SMD:R_0402_1005Metric, symbol Local_Device_Library:R1K
- added R3: R220K, Resistor_SMD:R_0603_1608Metric, symbol Local_Device_Library:R220K
- added R6: R2.2K, Resistor_SMD:R_0402_1005Metric, symbol Local_Device_Library:R2.2K
- added R8: R330K, Resistor_SMD:R_0603_1608Metric, symbol Local_Device_Library:R330K
- added RN1: 4_DIP_R4.7K, Local_Resistor_Library:RES-ARRAY-SMD_0603-8P-L3.2-W1.6-BL, symbol Local_Device_Library:4_DIP_R4.7K
- added SW5: SMD-SW-4_Tactile, Local_Misckllaneous_Library:SW_Tactile_Straight_(F.Mount), symbol Local_Miscellaneous_Library:SMD-SW-4_Tactile
- added U1: APKLVSR_OLEDM_0.96_I2C-IIC, Local_Misckllaneous_Library:APKLVSR_OLEDM_0.96_I2C-IIC, symbol Local_Miscellaneous_Library:APKLVSR_OLEDM_0.96_I2C-IIC
- C1, C7: JLCBCB Part https://jlcpcb.com/parts/componentSearch?isFirstLevel=true&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 -> https://jlcpcb.com/partdetail/20411-CL10A106KP8NNNC/C19702
- F1: footprint (none) -> Fuse:Fuseholder_Clip-5x20mm_Littelfuse_519_Inline_P20.60x5.00mm_D1.00mm_Horizontal; Excluded from BOM (none) -> YES; Mount Option (none) -> F.Mount; now left out of the parts list
- J7: renamed from J3; footprint (none) -> Local_Connectors:RJ14_Horizontal; Excluded from BOM (none) -> YES; Mount Option (none) -> F.Mount; now left out of the parts list
- J8: renamed from J1; footprint (none) -> TerminalBlock:TerminalBlock_MaiXu_MX126-5.0-02P_1x02_P5.00mm; Excluded from BOM (none) -> YES; Mount Option (none) -> F.Mount; now left out of the parts list
- R19: value 47K -> R2,1K; footprint (none) -> Local_Resistor_Library:R_Axial_DIN0207_L6.3mm_D2.5mm_P10.16mm_Horizontal; Excluded from BOM (none) -> YES; Famely (none) -> Resistors - THT; Mount Option (none) -> F.Mount; now left out of the parts list
- RV1: footprint (none) -> Varistor:RV_Disc_D15.5mm_W4.8mm_P7.5mm; Excluded from BOM (none) -> YES; Mount Option (none) -> F.Mount; now left out of the parts list
- SW1: footprint (none) -> Local_Switch_Library:SW_PUSH; Excluded from BOM (none) -> YES; Mount Option (none) -> F.Mount; now left out of the parts list
- SW2, SW3, SW4: footprint (none) -> Local_Switch_Library:SW_PUSH; Excluded from BOM (none) -> YES; now left out of the parts list
- U2: Mount Option (none) -> F.Mount
- renumbered U5 to U3, U1 to U3
Connections:
- net +3.3V: now also C1.1, C2.1, J5.1 (Pin_1), R15.1, R17.2
- net +3.3VA: now also J3.1 (Pin_1), U1.2 (VCC)
- net BASE_H: now also R10.2
- net DLY_H: now also C15.2, R4.1; no longer R19.2
- net Direct Reset GPIO: now also Q2.3 (C)
- net EDGE_H: now also D5.2 (A)
- net GND: now also J7.1, U2.13, U2.7 (GND), C10.2, C11.2, C12.2, C14.2, C16.2, C17.2, C18.2, C9.2, D6.2 (A), J5.4 (Pin_4), PS1.3 (-VOUT), Q1.2 (E), Q2.2 (E), Q3.2 (E), R11.2, R14.2, R16.2, R3.2, R5.2, R7.2, RN1.5 (R4.2), RN1.6 (R3.2), RN1.7 (R2.2), RN1.8 (R1.2)
- net GND1: now also J3.4 (Pin_4), SW5.1, SW5.2, U1.1 (GND)
- net HARD_RESET_GPIO: now also R13.1
- net Kill Switch: now also C12.1, C13.2, J4.6 (Pin_6), Q1.3 (C), R1.2
- net N250: now also C14.1, D5.1 (K), R3.1
- net N3S: now also C16.1, Q3.3 (C), R9.2
- net NSTART: now also C15.1, D6.1 (K), D7.2 (A), R5.1; no longer D4.1 (K)
- net NTRIG: now also D4.1 (K), C13.1, R2.2
- net OLED Touch: now also J4.5 (Pin_5)
- net SCL: now also J5.2 (Pin_2)
- net SDA: now also J5.3 (Pin_3)
- net START_H: now also R6.1
- net VCC: now also Q9.3 (D)
- net ext. LED1: now also R19.1, R20.1
- net ext. LED2: now also R18.1, R21.1
- net at F1.1, RV1.1: now also PS1.2 (VAC_IN(L))
- net at J8.2 (Pin_2), RV1.2: now also PS1.1 (VAC_IN(N))
- net at C5.2, U2.9: now also J4.3 (Pin_3), RN1.3 (R3.1)
- net at C3.2, U2.3: now also J4.1 (Pin_1), RN1.1 (R1.1)
- net at C4.2, U2.5: now also J4.2 (Pin_2), RN1.2 (R2.1)
- net at C6.2, U2.11: now also J4.4 (Pin_4), RN1.4 (R4.1)
- net at A1.4 (IO34_(no_pullup)): now also J2.1 (Pin_1)
- net at Q4.1 (B): now also R10.1, R11.1
- net at Q4.3 (C): now also Q9.1 (G), R12.2
- net at SW2.1: now also J1.2 (Pin_2)
- net at SW3.1: now also J1.3 (Pin_3)
- net at J7.3, U2.1: now also J7.4, C18.1, R17.1; no longer C2.1
- net at SW4.1: now also J1.4 (Pin_4)
- net +5V: now reaches U3.14 (VCC)
- net +5V: now also C10.1, C9.1, D7.1 (K), PS1.4 (+VOUT), Q9.2 (S), R1.1, R12.1, R2.1, R8.1
- net at SW1.1: now also J1.1 (Pin_1)
- net at D2.1 (K): now also J3.6 (Pin_6)
- net at D1.1 (K): now also J3.5 (Pin_5)
- new net: C17.1, J2.2 (Pin_2), R15.2, R16.1
- new net: C11.1, Q1.1 (B), R13.2, R14.1
- new net: Q3.1 (B), R6.2, R7.1
- new net: J3.2 (Pin_2), U1.3 (SCL)
- new net: J3.3 (Pin_3), U1.4 (SDA)
- new net: Q2.1 (B), R4.2
- new net: R8.2, R9.1
- new net: J1.5 (Pin_5), J6.1 (Pin_1)
- new net: J5.5 (Pin_5), R19.2, R20.2
- new net: J5.6 (Pin_6), R18.2, R21.2
- new net: J1.6 (Pin_6), SW5.3 (K), SW5.4 (A)
- no-connect marks 0 -> 14
Other:
- note added: "Keep near U2 pin 14"
- moved on the sheet: F1, J8, RV1, U2F, U2G, U3G

Commit message: HW: PCB revision 1.0.0
Parts:
- R14, R15, R16: footprint Resistor_SMD:R_0402_1005Metric -> Resistor_SMD:R_0805_2012Metric; JLCBCB Part https://jlcpcb.com/partdetail/26487-0402WGF1002TCE/C25744 -> https://jlcpcb.com/partdetail/18102-0805W8F1002T5E/C17414; JLCPCB Part # C25744 -> C17414; MFR. Part # 0402WGF1002TCE -> 0805W8F1002T5E; Package 0402 -> 0805
